Commit message: Merge in a batch of the changes from Stereolabs

File: urdf/zed.urdf (robot description, URDF)
Before this commit: robot zed_camera, 4 links, 3 joints
Links:
- removed link zed_center
- removed link zed_depth_camera
- removed link zed_left_camera
- removed link zed_right_camera
- added link zed_camera_center; visual mesh filename=package://zed_wrapper/urdf/ZED.stl
- added link zed_left_camera_frame
- added link zed_left_camera_optical_frame
- added link zed_right_camera_frame
- added link zed_right_camera_optical_frame
Joints:
- removed joint zed_depth_camera_joint
- added joint zed_left_camera_optical_joint: type fixed, parent zed_left_camera_frame, child zed_left_camera_optical_frame, origin xyz=0 0 0 rpy=-1.57079632679 0.0 -1.57079632679
- added joint zed_right_camera_optical_joint: type fixed, parent zed_right_camera_frame, child zed_right_camera_optical_frame, origin xyz=0 0 0 rpy=-1.57079632679 0.0 -1.57079632679
- joint zed_left_camera_joint: child zed_left_camera -> zed_left_camera_frame; parent zed_center -> zed_camera_center
- joint zed_right_camera_joint: child zed_right_camera -> zed_right_camera_frame; parent zed_center -> zed_camera_center
